File: hex_master_board/hex_master_board.sch (KiCad schematic (older format))
At the start: 40 parts

Commit message: Commit local changes from last semester
Parts:
- removed R? (x2): 1k, symbol Device:R
- added C3: 0.1uF, symbol Device:C
- added R17, R18, R19, R20, R21, R22, R7: 10k, symbol Device:R
- added R2, R3, R4, R5, R8: 1k, symbol Device:R
- added U2: 74LVC1G157GV_MUX2, hex_master_board:74LVC1G157_MUX2_TSOP6, symbol hex_master_sym:74LVC1G157GV_MUX2
- J1: renamed from J?; footprint (none) -> hex_master_board:USB micro 609-4616-1-ND
- U1: renamed from U?; footprint (none) -> hex_master_board:Jack_CP-002B-ND
- gave numbers to parts that had none: 36
Connections:
- net labels added: A0, A1, A2, A3, A4, A5, A6, A7, USB_RXD, USB_TXD, XBEE_RXD, XBEE_TXD
- wire segments 211 -> 248
Other:
- note added: "Internal pull-ups, D0-D5\n"
- note added: "Make sure using power as a \nlogic level isn't sketchy"
- note added: "Serial Multiplexing\n\n"
- note added: "Switch Inputs"

Commit message: Add placeholder switch symbols and TODO list in schematic
Parts:
- added SW? (x6): SW_DIP_x01, symbol Switch:SW_DIP_x01
Connections:
- wire segments 248 -> 245
Other:
- note added: "Reset\nButton"
- note added: "TODO spec and integrate an IMU that uses I2C\nTODO verify that serial mux won't break everything\nTODO actually spec connectors for foot limit switch wires\nTODO finish creating all footprints\nTODO make some high-level layout decisions\n"
- note added: "These are for switches on the hexapod feet\nInternal pull-ups, D0-D5\n"
- note removed: "Internal pull-ups, D0-D5\n"
Changed lines of the file:
@@
 	0    1    1    0
 $EndComp
-Wire Wire Line
-	4650 4900 4750 4900
 $Comp
 L Device:R R12
@@
 $EndComp
 Wire Wire Line
-	4750 4900 4750 4850
-Connection ~ 4750 4900
-Wire Wire Line
 	4750 3950 4750 3850
 $Comp
@@
 	1    0    0    -1
 $EndComp
-Wire Wire Line
-	4750 4850 4800 4850
-Wire Wire Line
-	4800 4850 4800 4900
-Connection ~ 4750 4850
-Wire Wire Line
-	4750 4250 4750 4850
 Wire Wire Line
 	3450 3550 3450 3650
@@
 	5850 6300 5850 6400
 Wire Wire Line
-	4800 4900 6100 4900
-Wire Wire Line
 	5800 5100 6400 5100
 Wire Wire Line
@@
 L hex_master_sym:Pushbutton_Stockroom U6
 U 1 1 5CBD5BFF
-P 4550 6050
-F 0 "U6" H 4550 6875 50  0000 C CNN
-F 1 "Pushbutton_Stockroom" H 4550 6784 50  0000 C CNN
-F 2 "" H 4550 6250 50  0001 C CNN
-F 3 "" H 4550 6250 50  0001 C CNN
-	1    4550 6050
-	1    0    0    -1
-$EndComp
-Wire Wire Line
-	4750 4900 4750 5450
-Wire Wire Line
-	4750 5750 4750 5850
-NoConn ~ 4350 5450
-NoConn ~ 4350 5750
+P 4200 7800
+F 0 "U6" H 4200 8625 50  0000 C CNN
+F 1 "Pushbutton_Stockroom" H 4200 8534 50  0000 C CNN
+F 2 "" H 4200 8000 50  0001 C CNN
+F 3 "" H 4200 8000 50  0001 C CNN
+	1    4200 7800
+	1    0    0    -1
+$EndComp
+Wire Wire Line
+	4400 7500 4400 7600
+NoConn ~ 4000 7200
+NoConn ~ 4000 7500
 $Comp
 L power:GND #PWR0127
 U 1 1 5CBEC62B
-P 4750 5850
-F 0 "#PWR0127" H 4750 5600 50  0001 C CNN
-F 1 "GND" H 4755 5677 50  0000 C CNN
-F 2 "" H 4750 5850 50  0001 C CNN
-F 3 "" H 4750 5850 50  0001 C CNN
-	1    4750 5850
+P 4400 7600
+F 0 "#PWR0127" H 4400 7350 50  0001 C CNN
+F 1 "GND" H 4405 7427 50  0000 C CNN
+F 2 "" H 4400 7600 50  0001 C CNN
+F 3 "" H 4400 7600 50  0001 C CNN
+	1    4400 7600
 	1    0    0    -1
 $EndComp
@@
 Wire Wire Line
 	6100 4900 6100 4750
-Connection ~ 6100 4900
 Wire Wire Line
 	6100 4900 6400 4900
@@
 Text Notes 8350 4700 0    138  ~ 0
 LED\n
-Text Notes 13550 1150 0    138  ~ 0
+Text Notes 13400 1050 0    138  ~ 0
 Switch Inputs
-Text Notes 13750 1250 0    50   ~ 0
-Internal pull-ups, D0-D5\n
+Text Notes 13400 1250 0    50   ~ 0
+These are for switches on the hexapod feet\nInternal pull-ups, D0-D5\n
 $Comp
 L Device:R R17
@@
 	1    0    0    -1
 $EndComp
-Wire Wire Line
-	13100 1950 13100 2100
-Wire Wire Line
-	13400 1950 13400 2100
-Wire Wire Line
-	13700 1950 13700 2100
-Wire Wire Line
-	14000 1950 14000 2100
-Wire Wire Line
-	14300 1950 14300 2100
-Wire Wire Line
-	14600 1950 14600 2100
 $Comp
 L power:+5V #PWR0144
@@
 Wire Wire Line
 	13400 1550 13700 1550
-Text Label 13100 2100 0    50   ~ 0
-D0
-Text Label 13400 2100 0    50   ~ 0
-D1
-Text Label 13700 2100 0    50   ~ 0
-D2
-Text Label 14000 2100 0    50   ~ 0
-D3
-Text Label 14300 2100 0    50   ~ 0
-D4
-Text Label 14600 2100 0    50   ~ 0
-D5
 Text Label 6400 6700 2    50   ~ 0
 A0
@@
 Text Notes 1250 8050 0    50   ~ 0
 Make sure using power as a \nlogic level isn't sketchy
+Wire Wire Line
+	13100 1950 13100 2250
+$Comp
+L Switch:SW_DIP_x01 SW?
+U 1 1 5D863B63
+P 13100 2550
+F 0 "SW?" V 13054 2680 50  0000 L CNN
+F 1 "SW_DIP_x01" V 13145 2680 50  0000 L CNN
+F 2 "" H 13100 2550 50  0001 C CNN
+F 3 "" H 13100 2550 50  0001 C CNN
+	1    13100 2550
+	0    1    1    0
+$EndComp
+$Comp
+L Switch:SW_DIP_x01 SW?
+U 1 1 5D863CF5
+P 13400 2550
+F 0 "SW?" V 13354 2680 50  0000 L CNN
+F 1 "SW_DIP_x01" V 13445 2680 50  0000 L CNN
+F 2 "" H 13400 2550 50  0001 C CNN
+F 3 "" H 13400 2550 50  0001 C CNN
+	1    13400 2550
+	0    1    1    0
+$EndComp
+$Comp
+L Switch:SW_DIP_x01 SW?
+U 1 1 5D873601
+P 13700 2550
+F 0 "SW?" V 13654 2680 50  0000 L CNN
+F 1 "SW_DIP_x01" V 13745 2680 50  0000 L CNN
+F 2 "" H 13700 2550 50  0001 C CNN
+F 3 "" H 13700 2550 50  0001 C CNN
+	1    13700 2550
+	0    1    1    0
+$EndComp
+$Comp
+L Switch:SW_DIP_x01 SW?
+U 1 1 5D882F0E
+P 14000 2550
+F 0 "SW?" V 13954 2680 50  0000 L CNN
+F 1 "SW_DIP_x01" V 14045 2680 50  0000 L CNN
+F 2 "" H 14000 2550 50  0001 C CNN
+F 3 "" H 14000 2550 50  0001 C CNN
+	1    14000 2550
+	0    1    1    0
+$EndComp
+$Comp
+L Switch:SW_DIP_x01 SW?
+U 1 1 5D89281A
+P 14300 2550
+F 0 "SW?" V 14254 2680 50  0000 L CNN
+F 1 "SW_DIP_x01" V 14345 2680 50  0000 L CNN
+F 2 "" H 14300 2550 50  0001 C CNN
+F 3 "" H 14300 2550 50  0001 C CNN
+	1    14300 2550
+	0    1    1    0
+$EndComp
+$Comp
+L Switch:SW_DIP_x01 SW?
+U 1 1 5D8A2129
+P 14600 2550
+F 0 "SW?" V 14554 2680 50  0000 L CNN
+F 1 "SW_DIP_x01" V 14645 2680 50  0000 L CNN
+F 2 "" H 14600 2550 50  0001 C CNN
+F 3 "" H 14600 2550 50  0001 C CNN
+	1    14600 2550
+	0    1    1    0
+$EndComp
+Wire Wire Line
+	13400 1950 13400 2250
+Wire Wire Line
+	13700 1950 13700 2250
+Wire Wire Line
+	14000 1950 14000 2250
+Wire Wire Line
+	14300 1950 14300 2250
+Wire Wire Line
+	14600 1950 14600 2250
+$Comp
+L power:GND #PWR?
+U 1 1 5D90FAE1
+P 13100 2850
+F 0 "#PWR?" H 13100 2600 50  0001 C CNN
+F 1 "GND" H 13105 2677 50  0000 C CNN
+F 2 "" H 13100 2850 50  0001 C CNN
+F 3 "" H 13100 2850 50  0001 C CNN
+	1    13100 2850
+	1    0    0    -1
+$EndComp
+$Comp
+L power:GND #PWR?
+U 1 1 5D91F305
+P 13400 2850
+F 0 "#PWR?" H 13400 2600 50  0001 C CNN
+F 1 "GND" H 13405 2677 50  0000 C CNN
+F 2 "" H 13400 2850 50  0001 C CNN
+F 3 "" H 13400 2850 50  0001 C CNN
+	1    13400 2850
+	1    0    0    -1
+$EndComp
+$Comp
+L power:GND #PWR?
+U 1 1 5D92EB29
+P 13700 2850
+F 0 "#PWR?" H 13700 2600 50  0001 C CNN
+F 1 "GND" H 13705 2677 50  0000 C CNN
+F 2 "" H 13700 2850 50  0001 C CNN
+F 3 "" H 13700 2850 50  0001 C CNN
+	1    13700 2850
+	1    0    0    -1
+$EndComp
+$Comp
+L power:GND #PWR?
+U 1 1 5D93E34D
+P 14000 2850
+F 0 "#PWR?" H 14000 2600 50  0001 C CNN
+F 1 "GND" H 14005 2677 50  0000 C CNN
+F 2 "" H 14000 2850 50  0001 C CNN
+F 3 "" H 14000 2850 50  0001 C CNN
+	1    14000 2850
+	1    0    0    -1
+$EndComp
+$Comp
+L power:GND #PWR?
+U 1 1 5D95D3CF
+P 14300 2850
+F 0 "#PWR?" H 14300 2600 50  0001 C CNN
+F 1 "GND" H 14305 2677 50  0000 C CNN
+F 2 "" H 14300 2850 50  0001 C CNN
+F 3 "" H 14300 2850 50  0001 C CNN
+	1    14300 2850
+	1    0    0    -1
+$EndComp
+$Comp
+L power:GND #PWR?
+U 1 1 5D96CBF3
+P 14600 2850
+F 0 "#PWR?" H 14600 2600 50  0001 C CNN
+F 1 "GND" H 14605 2677 50  0000 C CNN
+F 2 "" H 14600 2850 50  0001 C CNN
+F 3 "" H 14600 2850 50  0001 C CNN
+	1    14600 2850
+	1    0    0    -1
+$EndComp
+Text Label 13100 2100 0    50   ~ 0
+D0
+Text Label 13400 2100 0    50   ~ 0
+D1
+Text Label 13700 2100 0    50   ~ 0
+D2
+Text Label 14000 2100 0    50   ~ 0
+D3
+Text Label 14300 2100 0    50   ~ 0
+D4
+Text Label 14600 2100 0    50   ~ 0
+D5
+Text Notes 4500 7450 0    50   ~ 0
+Reset\nButton
+Text Label 4400 6750 0    50   ~ 0
+~RESET
+Wire Wire Line
+	4400 6750 4400 7200
+Wire Wire Line
+	6100 4900 4750 4900
+Connection ~ 6100 4900
+Wire Wire Line
+	4750 4250 4750 4900
+Connection ~ 4750 4900
+Wire Wire Line
+	4750 4900 4650 4900
+Text Notes 9400 4950 0    50   ~ 0
+TODO spec and integrate an IMU that uses I2C\nTODO verify that serial mux won't break everything\nTODO actually spec connectors for foot limit switch wires\nTODO finish creating all footprints\nTODO make some high-level layout decisions\n
 $EndSCHEMATC

Commit message: Change voltage regulator to one stocked by digikey
Parts:
- removed U3: MCP1700-5002E_SOT23, Package_TO_SOT_SMD:SOT-23, symbol Regulator_Linear:MCP1700-5002E_SOT23
- added U?: AP2210N-lin-reg, symbol hex_master_sym:AP2210N-lin-reg
- D4: value LED -> IO_LED
Other:
- note added: "Logic Power"
- note added: "TODO spec and integrate an IMU that uses I2C\nTODO verify that serial mux won't break everything\nTODO power LIDAR (is this just raspi usb?)\n\nTODO actually spec connectors for foot limit switch wires\nTODO finish creating all footprints\nTODO make some high-level layout decisions\nTODO figure out arduino raspi communication\n"
- note removed: "TODO spec and integrate an IMU that uses I2C\nTODO verify that serial mux won't break everything\nTODO actually spec connectors for foot limit switch wires\nTODO finish creating all footprints\nTODO make some high-level layout decisions\n"
Changed lines of the file:
@@
 L hex_master_sym:Jack_CP-002B-ND U1
 U 1 1 5CB747C3
-P 1450 1550
-F 0 "U1" H 1506 2115 50  0000 C CNN
-F 1 "Jack_CP-002B-ND" H 1506 2024 50  0000 C CNN
-F 2 "hex_master_board:Jack_CP-002B-ND" H 1450 1500 50  0001 C CNN
-F 3 "" H 1450 1500 50  0001 C CNN
-	1    1450 1550
-	1    0    0    -1
-$EndComp
-$Comp
-L Regulator_Linear:MCP1700-5002E_SOT23 U3
-U 1 1 5CB7486F
-P 2800 1250
-F 0 "U3" H 2800 1492 50  0000 C CNN
-F 1 "MCP1700-5002E_SOT23" H 2800 1401 50  0000 C CNN
-F 2 "Package_TO_SOT_SMD:SOT-23" H 2800 1475 50  0001 C CNN
-F 3 "http://ww1.microchip.com/downloads/en/DeviceDoc/20001826C.pdf" H 2800 1250 50  0001 C CNN
-	1    2800 1250
-	1    0    0    -1
-$EndComp
-Wire Wire Line
-	1700 1250 2350 1250
+P 1050 1550
+F 0 "U1" H 1106 2115 50  0000 C CNN
+F 1 "Jack_CP-002B-ND" H 1106 2024 50  0000 C CNN
+F 2 "hex_master_board:Jack_CP-002B-ND" H 1050 1500 50  0001 C CNN
+F 3 "" H 1050 1500 50  0001 C CNN
+	1    1050 1550
+	1    0    0    -1
+$EndComp
+Wire Wire Line
+	1300 1250 1950 1250
 $Comp
 L hex_master_sym:TPS2113A U5
@@
 	1    0    0    -1
 $EndComp
-Wire Wire Line
-	3100 1250 3200 1250
 $Comp
 L Device:R R9
@@
 L power:GND #PWR0111
 U 1 1 5CB7F824
-P 2800 1800
-F 0 "#PWR0111" H 2800 1550 50  0001 C CNN
-F 1 "GND" H 2805 1627 50  0000 C CNN
-F 2 "" H 2800 1800 50  0001 C CNN
-F 3 "" H 2800 1800 50  0001 C CNN
-	1    2800 1800
+P 2550 1950
+F 0 "#PWR0111" H 2550 1700 50  0001 C CNN
+F 1 "GND" H 2555 1777 50  0000 C CNN
+F 2 "" H 2550 1950 50  0001 C CNN
+F 3 "" H 2550 1950 50  0001 C CNN
+	1    2550 1950
 	1    0    0    -1
 $EndComp
@@
 L power:GND #PWR0112
 U 1 1 5CB7F85E
-P 2350 1800
-F 0 "#PWR0112" H 2350 1550 50  0001 C CNN
-F 1 "GND" H 2355 1627 50  0000 C CNN
-F 2 "" H 2350 1800 50  0001 C CNN
-F 3 "" H 2350 1800 50  0001 C CNN
-	1    2350 1800
+P 1950 1800
+F 0 "#PWR0112" H 1950 1550 50  0001 C CNN
+F 1 "GND" H 1955 1627 50  0000 C CNN
+F 2 "" H 1950 1800 50  0001 C CNN
+F 3 "" H 1950 1800 50  0001 C CNN
+	1    1950 1800
 	1    0    0    -1
 $EndComp
@@
 L Device:C C1
 U 1 1 5CB7F8A6
-P 2350 1500
-F 0 "C1" H 2465 1546 50  0000 L CNN
-F 1 "1uF" H 2465 1455 50  0000 L CNN
-F 2 "" H 2388 1350 50  0001 C CNN
-F 3 "~" H 2350 1500 50  0001 C CNN
-	1    2350 1500
-	1    0    0    -1
-$EndComp
-Wire Wire Line
-	2350 1350 2350 1250
-Connection ~ 2350 1250
-Wire Wire Line
-	2350 1250 2500 1250
-Wire Wire Line
-	2350 1650 2350 1800
-Wire Wire Line
-	2800 1550 2800 1800
+P 1950 1500
+F 0 "C1" H 2065 1546 50  0000 L CNN
+F 1 "1uF" H 2065 1455 50  0000 L CNN
+F 2 "" H 1988 1350 50  0001 C CNN
+F 3 "~" H 1950 1500 50  0001 C CNN
+	1    1950 1500
+	1    0    0    -1
+$EndComp
+Wire Wire Line
+	1950 1350 1950 1250
+Connection ~ 1950 1250
+Wire Wire Line
+	1950 1650 1950 1800
 $Comp
 L power:GND #PWR0113
 U 1 1 5CB8188E
-P 1800 1600
-F 0 "#PWR0113" H 1800 1350 50  0001 C CNN
-F 1 "GND" H 1805 1427 50  0000 C CNN
-F 2 "" H 1800 1600 50  0001 C CNN
-F 3 "" H 1800 1600 50  0001 C CNN
-	1    1800 1600
-	1    0    0    -1
-$EndComp
-Wire Wire Line
-	1700 1450 1800 1450
-Wire Wire Line
-	1800 1450 1800 1600
+P 1400 1600
+F 0 "#PWR0113" H 1400 1350 50  0001 C CNN
+F 1 "GND" H 1405 1427 50  0000 C CNN
+F 2 "" H 1400 1600 50  0001 C CNN
+F 3 "" H 1400 1600 50  0001 C CNN
+	1    1400 1600
+	1    0    0    -1
+$EndComp
+Wire Wire Line
+	1300 1450 1400 1450
+Wire Wire Line
+	1400 1450 1400 1600
 $Comp
 L Interface_USB:FT232RL U4
@@
 P 8050 4450
 F 0 "D4" V 8088 4333 50  0000 R CNN
-F 1 "LED" V 7997 4333 50  0000 R CNN
+F 1 "IO_LED" V 7997 4333 50  0000 R CNN
 F 2 "" H 8050 4450 50  0001 C CNN
 F 3 "~" H 8050 4450 50  0001 C CNN
@@
 	1    0    0    -1
 $EndComp
-Text Notes 8350 4700 0    138  ~ 0
+Text Notes 8350 4800 0    138  ~ 0
 LED\n
 Text Notes 13400 1050 0    138  ~ 0
@@
 	4750 4900 4650 4900
 Text Notes 9400 4950 0    50   ~ 0
-TODO spec and integrate an IMU that uses I2C\nTODO verify that serial mux won't break everything\nTODO actually spec connectors for foot limit switch wires\nTODO finish creating all footprints\nTODO make some high-level layout decisions\n
+TODO spec and integrate an IMU that uses I2C\nTODO verify that serial mux won't break everything\nTODO power LIDAR (is this just raspi usb?)\n\nTODO actually spec connectors for foot limit switch wires\nTODO finish creating all footprints\nTODO make some high-level layout decisions\nTODO figure out arduino raspi communication\n
+Text Notes 750  1700 0    50   ~ 0
+Logic Power
+$Comp
+L hex_master_sym:AP2210N-lin-reg U?
+U 1 1 5D8C65D8
+P 2550 1000
+F 0 "U?" H 2550 1065 50  0000 C CNN
+F 1 "AP2210N-lin-reg" H 2550 974 50  0000 C CNN
+F 2 "" H 2550 1000 50  0001 C CNN
+F 3 "" H 2550 1000 50  0001 C CNN
+	1    2550 1000
+	1    0    0    -1
+$EndComp
+Wire Wire Line
+	2950 1250 3200 1250
+Wire Wire Line
+	2550 1650 2550 1950
+Wire Wire Line
+	1950 1250 2150 1250
 $EndSCHEMATC

Commit message: Added servo outs to schematic
Parts:
- added U?: Jack_CP-002B-ND, symbol hex_master_sym:Jack_CP-002B-ND
- added U? (x32): Servo_connector, symbol hex_master_sym:Servo_connector
- U?: footprint (none) -> Package_TO_SOT_SMD:SOT-23
Connections:
- net labels added: servo_power
- wire segments 245 -> 344
Other:
- note added: "Servo Ports\n"

Commit message: Add additional switch inputs
Parts:
- added R? (x6): 10k, symbol Device:R
- added SW? (x6): SW_DIP_x01, symbol Switch:SW_DIP_x01
- added U? (x4): EXB-2HV221JV, symbol hex_master_sym:EXB-2HV221JV
- R1, R6: value 1k -> 1kΩ
- R13: value R -> 350Ω
- U?: value AP2210N-lin-reg -> AP2210N-5.0TRG1-lin-reg
Connections:
- net labels added: D10, D11, D8, D9
- wire segments 344 -> 385
Other:
- note added: "TODOs are probably out of date, check Asana\n\nTODO spec and integrate an IMU that uses I2C\nTODO verify that serial mux won't break everything\nTODO power LIDAR (is this just raspi usb?)\n\nTODO actually spec connectors for foot limit switch wires\nTODO finish creating all footprints\nTODO make some high-level layout decisions\nTODO figure out arduino raspi communication\n"
- note removed: "TODO spec and integrate an IMU that uses I2C\nTODO verify that serial mux won't break everything\nTODO power LIDAR (is this just raspi usb?)\n\nTODO actually spec connectors for foot limit switch wires\nTODO finish creating all footprints\nTODO make some high-level layout decisions\nTODO figure out arduino raspi communication\n"

Commit message: Add footprints to resistors, capacitors, switch inputs
Parts:
- C1, C10, C11, C14, C15, C2, C3, C4, C5, C6, C7, C8, C9: footprint (none) -> Capacitor_SMD:C_0805_2012Metric_Pad1.15x1.40mm_HandSolder
- R1, R10, R11, R12, R15, R17, R18, R19, R2, R20, R21, R22, R3, R4, R5, R6, R7, R8, R9: footprint (none) -> Resistor_SMD:R_0805_2012Metric_Pad1.15x1.40mm_HandSolder
- R13: value 350Ω -> 1kΩ; footprint (none) -> Resistor_SMD:R_0805_2012Metric_Pad1.15x1.40mm_HandSolder
- R14, R16: value 4.7k -> 10k; footprint (none) -> Resistor_SMD:R_0805_2012Metric_Pad1.15x1.40mm_HandSolder
- R23, R24, R25, R26, R27, R28: renamed from R?; footprint (none) -> Resistor_SMD:R_0805_2012Metric_Pad1.15x1.40mm_HandSolder
- U10, U11, U29, U30: renamed from U?; footprint (none) -> hex_master_board:EXB-2HV221JV
- U12: renamed from U?; footprint (none) -> hex_master_board:Jack_CP-002B-ND
- U13, U14, U15, U16, U17, U18, U19, U20, U21, U22, U23, U24, U25, U26, U27, U28, U31, U32, U33, U34, U35, U36, U37, U38, U39, U40, U41, U42, U43, U44, U45, U46: renamed from U?; footprint (none) -> hex_master_board:servo_header
- gave numbers to parts that had none: 13
Connections:
- net labels added: D12
- wire segments 385 -> 394
Other:
- note added: "Comm LEDs\n"

Commit message: Add IO header symbol
Parts:
- added C?: 10uF, Capacitor_SMD:C_0805_2012Metric_Pad1.15x1.40mm_HandSolder, symbol Device:C
- added U? (x3): header_0.1_8, symbol hex_master_sym:header_0.1_8
Connections:
- net labels added: D13, D14, D15, D16, D17, D18, D19, D20, D21, D22, D23, D24, D25, D26, ~RX_LED, ~TX_LED
- net labels removed: D12, ~RX, ~TX
- wire segments 394 -> 407
- no-connect marks 16 -> 31
Other:
- note added: "FT232RQ"
- note added: "IO Breakouts"

Commit message: Add footprint for ICSP header, associate footprint for switch inputs
Parts:
- added U?: ICSP_breakout, symbol hex_master_sym:ICSP_breakout
- U? (x3): footprint (none) -> hex_master_board:header_0.1_8x
Connections:
- wire segments 407 -> 418
Other:
- note added: "ICSP Headers"
Changed lines of the file:
@@
 $EndComp
 NoConn ~ 4150 5200
-Text Label 7600 5900 0    50   ~ 0
+Text Label 7650 5900 0    50   ~ 0
 SCK
-Text Label 7600 6100 0    50   ~ 0
+Text Label 7650 6100 0    50   ~ 0
 MISO
-Text Label 7600 6000 0    50   ~ 0
+Text Label 7650 6000 0    50   ~ 0
 MOSI
 Wire Wire Line
@@
 F 0 "U?" H 5545 9178 50  0000 C CNN
 F 1 "header_0.1_8" H 5545 9087 50  0000 C CNN
-F 2 "" H 5550 9200 50  0001 C CNN
+F 2 "hex_master_board:header_0.1_8x" H 5550 9200 50  0001 C CNN
 F 3 "" H 5550 9200 50  0001 C CNN
 	1    5550 9600
@@
 F 0 "U?" H 6545 9178 50  0000 C CNN
 F 1 "header_0.1_8" H 6545 9087 50  0000 C CNN
-F 2 "" H 6550 9200 50  0001 C CNN
+F 2 "hex_master_board:header_0.1_8x" H 6550 9200 50  0001 C CNN
 F 3 "" H 6550 9200 50  0001 C CNN
 	1    6550 9600
@@
 F 0 "U?" H 7545 9178 50  0000 C CNN
 F 1 "header_0.1_8" H 7545 9087 50  0000 C CNN
-F 2 "" H 7550 9200 50  0001 C CNN
+F 2 "hex_master_board:header_0.1_8x" H 7550 9200 50  0001 C CNN
 F 3 "" H 7550 9200 50  0001 C CNN
 	1    7550 9600
@@
 NoConn ~ 6300 9750
 NoConn ~ 7600 6500
+Wire Wire Line
+	7650 5900 7600 5900
+Wire Wire Line
+	7600 6000 7650 6000
+Wire Wire Line
+	7650 6100 7600 6100
+$Comp
+L hex_master_sym:ICSP_breakout U?
+U 1 1 5DB051F0
+P 5150 8750
+F 0 "U?" H 5150 8975 50  0000 C CNN
+F 1 "ICSP_breakout" H 5150 8884 50  0000 C CNN
+F 2 "" H 5150 8900 50  0001 C CNN
+F 3 "" H 5150 8900 50  0001 C CNN
+	1    5150 8750
+	1    0    0    -1
+$EndComp
+$Comp
+L power:+5V #PWR?
+U 1 1 5DB05A40
+P 5600 8650
+F 0 "#PWR?" H 5600 8500 50  0001 C CNN
+F 1 "+5V" H 5615 8823 50  0000 C CNN
+F 2 "" H 5600 8650 50  0001 C CNN
+F 3 "" H 5600 8650 50  0001 C CNN
+	1    5600 8650
+	1    0    0    -1
+$EndComp
+Wire Wire Line
+	5500 8750 5600 8750
+Wire Wire Line
+	5600 8750 5600 8650
+$Comp
+L power:GND #PWR?
+U 1 1 5DB32C63
+P 5600 9050
+F 0 "#PWR?" H 5600 8800 50  0001 C CNN
+F 1 "GND" H 5605 8877 50  0000 C CNN
+F 2 "" H 5600 9050 50  0001 C CNN
+F 3 "" H 5600 9050 50  0001 C CNN
+	1    5600 9050
+	1    0    0    -1
+$EndComp
+Wire Wire Line
+	5500 8950 5600 8950
+Wire Wire Line
+	5600 8950 5600 9050
+Text Label 5550 8850 0    50   ~ 0
+MOSI
+Text Label 4750 8750 2    50   ~ 0
+MISO
+Text Label 4750 8850 2    50   ~ 0
+SCK
+Text Label 4750 8950 2    50   ~ 0
+~RESET
+Wire Wire Line
+	4750 8750 4800 8750
+Wire Wire Line
+	4750 8850 4800 8850
+Wire Wire Line
+	4750 8950 4800 8950
+Wire Wire Line
+	5500 8850 5550 8850
+Text Notes 4550 8300 0    118  ~ 0
+ICSP Headers
 $EndSCHEMATC
