File: hex_master_board/hex_master_board.sch (KiCad schematic (older format))
At the start: 112 parts, among them J1 USB_B_Micro, SW1 SW_DIP_x01, SW10 SW_DIP_x01, SW11 SW_DIP_x01, SW12 SW_DIP_x01, SW2 SW_DIP_x01, SW3 SW_DIP_x01, SW4 SW_DIP_x01, SW5 SW_DIP_x01, SW6 SW_DIP_x01, SW7 SW_DIP_x01, SW8 SW_DIP_x01, SW9 SW_DIP_x01, U1 Jack_CP-002B-ND, U10 EXB-2HV221JV, U11 EXB-2HV221JV, U12 Jack_CP-002B-ND, U13 Servo_connector, U14 Servo_connector, U15 Servo_connector, U16 Servo_connector, U17 Servo_connector, U18 Servo_connector, U19 Servo_connector, U2 74LVC1G157GV_MUX2, U20 Servo_connector, U21 Servo_connector, U22 Servo_connector, U23 Servo_connector, U24 Servo_connector, U25 Servo_connector, U26 Servo_connector, U27 Servo_connector, U28 Servo_connector, U29 EXB-2HV221JV, U3 AP2210N-5.0TRG1-lin-reg, U30 EXB-2HV221JV, U31 Servo_connector, U32 Servo_connector, U33 Servo_connector, U34 Servo_connector, U35 Servo_connector, U36 Servo_connector, U37 Servo_connector, U38 Servo_connector, U39 Servo_connector, U4 FT232RL, U40 Servo_connector, U41 Servo_connector, U42 Servo_connector, U43 Servo_connector, U44 Servo_connector, U45 Servo_connector, U46 Servo_connector, U5 TPS2113A, U6 Pushbutton_Stockroom, U7 ATmega2561-16AU, U8 PCA9685PW, U9 PCA9685PW, Y1 Crystal

Commit message: Start PCB layout!
Parts:
- D1, D2, D3, D4: footprint (none) -> hex_master_board:LED_SMD_1206
- R12, R15: footprint Resistor_SMD:R_0805_2012Metric_Pad1.15x1.40mm_HandSolder -> (none)
- SW1, SW10, SW11, SW12, SW2, SW3, SW4, SW5, SW6, SW7, SW8, SW9: footprint (none) -> hex_master_board:switch_ins
- gave numbers to parts that had none: 5
Other:
- note added: "Hexapod Control Board V0 --- DRAFT"

Commit message: Footprint for crystal, develop footprint further
Parts:
- C12, C13: footprint (none) -> Capacitor_SMD:C_0805_2012Metric_Pad1.15x1.40mm_HandSolder
- R12, R15: footprint (none) -> Resistor_SMD:R_0805_2012Metric_Pad1.15x1.40mm_HandSolder
- U47: footprint (none) -> hex_master_board:ICSP_header_0.1
- U6: footprint (none) -> hex_master_board:Pushbutton_Stockroom
- Y1: footprint (none) -> hex_master_board:Crystal_osc_535-10226-1-ND
Changed lines of the file:
@@
 F 0 "R12" H 4820 4146 50  0000 L CNN
 F 1 "1k" H 4820 4055 50  0000 L CNN
-F 2 "" V 4680 4100 50  0001 C CNN
+F 2 "Resistor_SMD:R_0805_2012Metric_Pad1.15x1.40mm_HandSolder" V 4680 4100 50  0001 C CNN
 F 3 "~" H 4750 4100 50  0001 C CNN
 	1    4750 4100
@@
 F 0 "C13" H 7365 4246 50  0000 L CNN
 F 1 "0.1uF" H 7365 4155 50  0000 L CNN
-F 2 "" H 7288 4050 50  0001 C CNN
+F 2 "Capacitor_SMD:C_0805_2012Metric_Pad1.15x1.40mm_HandSolder" H 7288 4050 50  0001 C CNN
 F 3 "~" H 7250 4200 50  0001 C CNN
 	1    7250 4200
@@
 F 0 "C12" H 6765 4246 50  0000 L CNN
 F 1 "0.1uF" H 6765 4155 50  0000 L CNN
-F 2 "" H 6688 4050 50  0001 C CNN
+F 2 "Capacitor_SMD:C_0805_2012Metric_Pad1.15x1.40mm_HandSolder" H 6688 4050 50  0001 C CNN
 F 3 "~" H 6650 4200 50  0001 C CNN
 	1    6650 4200
@@
 F 0 "Y1" V 5454 5331 50  0000 L CNN
 F 1 "Crystal" V 5545 5331 50  0000 L CNN
-F 2 "" H 5500 5200 50  0001 C CNN
+F 2 "hex_master_board:Crystal_osc_535-10226-1-ND" H 5500 5200 50  0001 C CNN
 F 3 "~" H 5500 5200 50  0001 C CNN
 	1    5500 5200
@@
 F 0 "U6" H 4200 8625 50  0000 C CNN
 F 1 "Pushbutton_Stockroom" H 4200 8534 50  0000 C CNN
-F 2 "" H 4200 8000 50  0001 C CNN
+F 2 "hex_master_board:Pushbutton_Stockroom" H 4200 8000 50  0001 C CNN
 F 3 "" H 4200 8000 50  0001 C CNN
 	1    4200 7800
@@
 F 0 "R15" H 8120 4896 50  0000 L CNN
 F 1 "1k" H 8120 4805 50  0000 L CNN
-F 2 "" V 7980 4850 50  0001 C CNN
+F 2 "Resistor_SMD:R_0805_2012Metric_Pad1.15x1.40mm_HandSolder" V 7980 4850 50  0001 C CNN
 F 3 "~" H 8050 4850 50  0001 C CNN
 	1    8050 4850
@@
 F 0 "U47" H 5150 8975 50  0000 C CNN
 F 1 "ICSP_breakout" H 5150 8884 50  0000 C CNN
-F 2 "" H 5150 8900 50  0001 C CNN
+F 2 "hex_master_board:ICSP_header_0.1" H 5150 8900 50  0001 C CNN
 F 3 "" H 5150 8900 50  0001 C CNN
 	1    5150 8750

Commit message: More progress on layout
Parts:
- removed U48: header_0.1_8, hex_master_board:header_0.1_8x, symbol hex_master_sym:header_0.1_8
- added U48: header_0.1_8_powered, hex_master_board:header_0.1_8_power, symbol hex_master_sym:header_0.1_8_powered
Connections:
- wire segments 418 -> 422
Changed lines of the file:
@@
 Text Notes 3200 5200 0    50   ~ 0
 FT232RQ
-$Comp
-L hex_master_sym:header_0.1_8 U48
-U 1 1 5DD239EE
-P 5550 9600
-F 0 "U48" H 5545 9178 50  0000 C CNN
-F 1 "header_0.1_8" H 5545 9087 50  0000 C CNN
-F 2 "hex_master_board:header_0.1_8x" H 5550 9200 50  0001 C CNN
-F 3 "" H 5550 9200 50  0001 C CNN
-	1    5550 9600
-	1    0    0    -1
-$EndComp
-Text Label 5900 9650 1    50   ~ 0
+Text Label 5600 9600 1    50   ~ 0
 A0
-Text Label 5800 9650 1    50   ~ 0
+Text Label 5500 9600 1    50   ~ 0
 A1
-Text Label 5700 9650 1    50   ~ 0
+Text Label 5400 9600 1    50   ~ 0
 A2
-Text Label 5600 9650 1    50   ~ 0
+Text Label 5300 9600 1    50   ~ 0
 A3
-Text Label 5500 9650 1    50   ~ 0
+Text Label 5200 9600 1    50   ~ 0
 A4
-Text Label 5400 9650 1    50   ~ 0
+Text Label 5100 9600 1    50   ~ 0
 A5
-Text Label 5300 9650 1    50   ~ 0
+Text Label 5000 9600 1    50   ~ 0
 A6
-Text Label 5200 9650 1    50   ~ 0
+Text Label 4900 9600 1    50   ~ 0
 A7
 Wire Wire Line
-	5200 9650 5200 9750
-Wire Wire Line
-	5300 9750 5300 9650
-Wire Wire Line
-	5400 9650 5400 9750
-Wire Wire Line
-	5500 9750 5500 9650
-Wire Wire Line
-	5600 9650 5600 9750
-Wire Wire Line
-	5700 9750 5700 9650
-Wire Wire Line
-	5800 9650 5800 9750
-Wire Wire Line
-	5900 9750 5900 9650
+	4900 9600 4900 9700
+Wire Wire Line
+	5000 9700 5000 9600
+Wire Wire Line
+	5100 9600 5100 9700
+Wire Wire Line
+	5200 9700 5200 9600
+Wire Wire Line
+	5300 9600 5300 9700
+Wire Wire Line
+	5400 9700 5400 9600
+Wire Wire Line
+	5500 9600 5500 9700
+Wire Wire Line
+	5600 9700 5600 9600
 Text Notes 5100 10600 0    118  ~ 0
 IO Breakouts
@@
 Text Notes 12050 10300 0    106  ~ 0
 Hexapod Control Board V0 --- DRAFT
+$Comp
+L hex_master_sym:header_0.1_8_powered U48
+U 1 1 5DBAE69B
+P 5250 9550
+F 0 "U48" H 5250 9028 50  0000 C CNN
+F 1 "header_0.1_8_powered" H 5250 8937 50  0000 C CNN
+F 2 "hex_master_board:header_0.1_8_power" H 5250 9150 50  0001 C CNN
+F 3 "" H 5250 9150 50  0001 C CNN
+	1    5250 9550
+	1    0    0    -1
+$EndComp
+$Comp
+L power:GND #PWR0197
+U 1 1 5DBDC669
+P 5850 10000
+F 0 "#PWR0197" H 5850 9750 50  0001 C CNN
+F 1 "GND" H 5855 9827 50  0000 C CNN
+F 2 "" H 5850 10000 50  0001 C CNN
+F 3 "" H 5850 10000 50  0001 C CNN
+	1    5850 10000
+	1    0    0    -1
+$EndComp
+$Comp
+L power:+5V #PWR0198
+U 1 1 5DBDC780
+P 4650 9850
+F 0 "#PWR0198" H 4650 9700 50  0001 C CNN
+F 1 "+5V" H 4665 10023 50  0000 C CNN
+F 2 "" H 4650 9850 50  0001 C CNN
+F 3 "" H 4650 9850 50  0001 C CNN
+	1    4650 9850
+	1    0    0    -1
+$EndComp
+Wire Wire Line
+	4700 9950 4650 9950
+Wire Wire Line
+	4650 9950 4650 9850
+Wire Wire Line
+	5800 9950 5850 9950
+Wire Wire Line
+	5850 9950 5850 10000
 $EndSCHEMATC

Commit message: Add accelerometer, more tracing
Parts:
- added U51: LIS3DH_breakout, hex_master_board:LIS3DH_IMU_BOARD, symbol hex_master_sym:LIS3DH_breakout
Connections:
- wire segments 422 -> 426
- no-connect marks 31 -> 38
Other:
- note added: "Accelerometer"
- note added: "Communicates with Atmega\nover I2C\n"
Changed lines of the file:
@@
 Wire Wire Line
 	5850 9950 5850 10000
+$Comp
+L hex_master_sym:LIS3DH_breakout U51
+U 1 1 5DC27FDC
+P 9650 4150
+F 0 "U51" H 10078 3996 50  0000 L CNN
+F 1 "LIS3DH_breakout" H 10078 3905 50  0000 L CNN
+F 2 "hex_master_board:LIS3DH_IMU_BOARD" H 9350 4050 50  0001 C CNN
+F 3 "" H 9350 4050 50  0001 C CNN
+	1    9650 4150
+	1    0    0    -1
+$EndComp
+Text Notes 10300 4000 0    138  ~ 0
+Accelerometer
+Text Notes 10300 4200 0    50   ~ 0
+Communicates with Atmega\nover I2C\n
+Text Label 9600 4650 3    50   ~ 0
+SCL
+Text Label 9700 4650 3    50   ~ 0
+SDA
+Wire Wire Line
+	9500 4650 9500 4900
+$Comp
+L power:GND #PWR0199
+U 1 1 5DC874A9
+P 9500 4900
+F 0 "#PWR0199" H 9500 4650 50  0001 C CNN
+F 1 "GND" H 9505 4727 50  0000 C CNN
+F 2 "" H 9500 4900 50  0001 C CNN
+F 3 "" H 9500 4900 50  0001 C CNN
+	1    9500 4900
+	1    0    0    -1
+$EndComp
+Wire Wire Line
+	9300 4650 9300 4700
+Wire Wire Line
+	9050 4700 9050 4500
+Wire Wire Line
+	9050 4700 9300 4700
+$Comp
+L power:+5V #PWR0200
+U 1 1 5DCB756C
+P 9050 4500
+F 0 "#PWR0200" H 9050 4350 50  0001 C CNN
+F 1 "+5V" H 9065 4673 50  0000 C CNN
+F 2 "" H 9050 4500 50  0001 C CNN
+F 3 "" H 9050 4500 50  0001 C CNN
+	1    9050 4500
+	1    0    0    -1
+$EndComp
+NoConn ~ 9400 4650
+NoConn ~ 9800 4650
+NoConn ~ 9900 4650
+NoConn ~ 10000 4650
+NoConn ~ 9550 4050
+NoConn ~ 9650 4050
+NoConn ~ 9750 4050
 $EndSCHEMATC

Commit message: Add I2C headers, fully connect board
Parts:
- added U52: header_0.1_I2C, hex_master_board:header_0.1_i2c_12, symbol hex_master_sym:header_0.1_I2C
Connections:
- wire segments 426 -> 430
Other:
- note removed: "TODOs are probably out of date, check Asana\n\nTODO spec and integrate an IMU that uses I2C\nTODO verify that serial mux won't break everything\nTODO power LIDAR (is this just raspi usb?)\n\nTODO actually spec connectors for foot limit switch wires\nTODO finish creating all footprints\nTODO make some high-level layout decisions\nTODO figure out arduino raspi communication\n"
Changed lines of the file:
@@
 Wire Wire Line
 	4750 4900 4650 4900
-Text Notes 9100 10700 0    50   ~ 0
-TODOs are probably out of date, check Asana\n\nTODO spec and integrate an IMU that uses I2C\nTODO verify that serial mux won't break everything\nTODO power LIDAR (is this just raspi usb?)\n\nTODO actually spec connectors for foot limit switch wires\nTODO finish creating all footprints\nTODO make some high-level layout decisions\nTODO figure out arduino raspi communication\n
 Text Notes 750  1700 0    50   ~ 0
 Logic Power
@@
 Text Notes 3200 5200 0    50   ~ 0
 FT232RQ
-Text Label 5600 9600 1    50   ~ 0
+Text Label 5200 9750 1    50   ~ 0
 A0
-Text Label 5500 9600 1    50   ~ 0
+Text Label 5100 9750 1    50   ~ 0
 A1
-Text Label 5400 9600 1    50   ~ 0
+Text Label 5000 9750 1    50   ~ 0
 A2
-Text Label 5300 9600 1    50   ~ 0
+Text Label 4900 9750 1    50   ~ 0
 A3
-Text Label 5200 9600 1    50   ~ 0
+Text Label 4800 9750 1    50   ~ 0
 A4
-Text Label 5100 9600 1    50   ~ 0
+Text Label 4700 9750 1    50   ~ 0
 A5
-Text Label 5000 9600 1    50   ~ 0
+Text Label 4600 9750 1    50   ~ 0
 A6
-Text Label 4900 9600 1    50   ~ 0
+Text Label 4500 9750 1    50   ~ 0
 A7
 Wire Wire Line
-	4900 9600 4900 9700
-Wire Wire Line
-	5000 9700 5000 9600
-Wire Wire Line
-	5100 9600 5100 9700
-Wire Wire Line
-	5200 9700 5200 9600
-Wire Wire Line
-	5300 9600 5300 9700
-Wire Wire Line
-	5400 9700 5400 9600
-Wire Wire Line
-	5500 9600 5500 9700
-Wire Wire Line
-	5600 9700 5600 9600
-Text Notes 5100 10600 0    118  ~ 0
+	4500 9750 4500 9850
+Wire Wire Line
+	4600 9850 4600 9750
+Wire Wire Line
+	4700 9750 4700 9850
+Wire Wire Line
+	4800 9850 4800 9750
+Wire Wire Line
+	4900 9750 4900 9850
+Wire Wire Line
+	5000 9850 5000 9750
+Wire Wire Line
+	5100 9750 5100 9850
+Wire Wire Line
+	5200 9850 5200 9750
+Text Notes 4700 10750 0    118  ~ 0
 IO Breakouts
 Text Label 6400 7800 2    50   ~ 0
@@
 L hex_master_sym:header_0.1_8 U49
 U 1 1 5E0A6DBA
-P 6550 9600
-F 0 "U49" H 6545 9178 50  0000 C CNN
-F 1 "header_0.1_8" H 6545 9087 50  0000 C CNN
-F 2 "hex_master_board:header_0.1_8x" H 6550 9200 50  0001 C CNN
-F 3 "" H 6550 9200 50  0001 C CNN
-	1    6550 9600
+P 6150 9750
+F 0 "U49" H 6145 9328 50  0000 C CNN
+F 1 "header_0.1_8" H 6145 9237 50  0000 C CNN
+F 2 "hex_master_board:header_0.1_8x" H 6150 9350 50  0001 C CNN
+F 3 "" H 6150 9350 50  0001 C CNN
+	1    6150 9750
 	1    0    0    -1
 $EndComp
@@
 L hex_master_sym:header_0.1_8 U50
 U 1 1 5E0D1B6D
-P 7550 9600
-F 0 "U50" H 7545 9178 50  0000 C CNN
-F 1 "header_0.1_8" H 7545 9087 50  0000 C CNN
-F 2 "hex_master_board:header_0.1_8x" H 7550 9200 50  0001 C CNN
-F 3 "" H 7550 9200 50  0001 C CNN
-	1    7550 9600
-	1    0    0    -1
-$EndComp
-Text Label 7900 9750 1    50   ~ 0
+P 7150 9750
+F 0 "U50" H 7145 9328 50  0000 C CNN
+F 1 "header_0.1_8" H 7145 9237 50  0000 C CNN
+F 2 "hex_master_board:header_0.1_8x" H 7150 9350 50  0001 C CNN
+F 3 "" H 7150 9350 50  0001 C CNN
+	1    7150 9750
+	1    0    0    -1
+$EndComp
+Text Label 7500 9900 1    50   ~ 0
 D13
-Text Label 7800 9750 1    50   ~ 0
+Text Label 7400 9900 1    50   ~ 0
 D14
-Text Label 7700 9750 1    50   ~ 0
+Text Label 7300 9900 1    50   ~ 0
 D15
-Text Label 7600 9750 1    50   ~ 0
+Text Label 7200 9900 1    50   ~ 0
 D16
-Text Label 7500 9750 1    50   ~ 0
+Text Label 7100 9900 1    50   ~ 0
 D17
-Text Label 7400 9750 1    50   ~ 0
+Text Label 7000 9900 1    50   ~ 0
 D18
-Text Label 7300 9750 1    50   ~ 0
+Text Label 6900 9900 1    50   ~ 0
 D19
-Text Label 7200 9750 1    50   ~ 0
+Text Label 6800 9900 1    50   ~ 0
 D20
-Text Label 6900 9750 1    50   ~ 0
+Text Label 6500 9900 1    50   ~ 0
 D21
-Text Label 6800 9750 1    50   ~ 0
+Text Label 6400 9900 1    50   ~ 0
 D22
-Text Label 6700 9750 1    50   ~ 0
+Text Label 6300 9900 1    50   ~ 0
 D23
-Text Label 6600 9750 1    50   ~ 0
+Text Label 6200 9900 1    50   ~ 0
 D24
-Text Label 6500 9750 1    50   ~ 0
+Text Label 6100 9900 1    50   ~ 0
 D25
-Text Label 6400 9750 1    50   ~ 0
+Text Label 6000 9900 1    50   ~ 0
 D26
-NoConn ~ 6200 9750
-NoConn ~ 6300 9750
+NoConn ~ 5800 9900
+NoConn ~ 5900 9900
 NoConn ~ 7600 6500
 Wire Wire Line
@@
 L hex_master_sym:header_0.1_8_powered U48
 U 1 1 5DBAE69B
-P 5250 9550
-F 0 "U48" H 5250 9028 50  0000 C CNN
-F 1 "header_0.1_8_powered" H 5250 8937 50  0000 C CNN
-F 2 "hex_master_board:header_0.1_8_power" H 5250 9150 50  0001 C CNN
-F 3 "" H 5250 9150 50  0001 C CNN
-	1    5250 9550
+P 4850 9700
+F 0 "U48" H 4850 9178 50  0000 C CNN
+F 1 "header_0.1_8_powered" H 4850 9087 50  0000 C CNN
+F 2 "hex_master_board:header_0.1_8_power" H 4850 9300 50  0001 C CNN
+F 3 "" H 4850 9300 50  0001 C CNN
+	1    4850 9700
 	1    0    0    -1
 $EndComp
@@
 L power:GND #PWR0197
 U 1 1 5DBDC669
-P 5850 10000
-F 0 "#PWR0197" H 5850 9750 50  0001 C CNN
-F 1 "GND" H 5855 9827 50  0000 C CNN
-F 2 "" H 5850 10000 50  0001 C CNN
-F 3 "" H 5850 10000 50  0001 C CNN
-	1    5850 10000
+P 5450 10150
+F 0 "#PWR0197" H 5450 9900 50  0001 C CNN
+F 1 "GND" H 5455 9977 50  0000 C CNN
+F 2 "" H 5450 10150 50  0001 C CNN
+F 3 "" H 5450 10150 50  0001 C CNN
+	1    5450 10150
 	1    0    0    -1
 $EndComp
@@
 L power:+5V #PWR0198
 U 1 1 5DBDC780
-P 4650 9850
-F 0 "#PWR0198" H 4650 9700 50  0001 C CNN
-F 1 "+5V" H 4665 10023 50  0000 C CNN
-F 2 "" H 4650 9850 50  0001 C CNN
-F 3 "" H 4650 9850 50  0001 C CNN
-	1    4650 9850
-	1    0    0    -1
-$EndComp
-Wire Wire Line
-	4700 9950 4650 9950
-Wire Wire Line
-	4650 9950 4650 9850
-Wire Wire Line
-	5800 9950 5850 9950
-Wire Wire Line
-	5850 9950 5850 10000
+P 4250 10000
+F 0 "#PWR0198" H 4250 9850 50  0001 C CNN
+F 1 "+5V" H 4265 10173 50  0000 C CNN
+F 2 "" H 4250 10000 50  0001 C CNN
+F 3 "" H 4250 10000 50  0001 C CNN
+	1    4250 10000
+	1    0    0    -1
+$EndComp
+Wire Wire Line
+	4300 10100 4250 10100
+Wire Wire Line
+	4250 10100 4250 10000
+Wire Wire Line
+	5400 10100 5450 10100
+Wire Wire Line
+	5450 10100 5450 10150
 $Comp
 L hex_master_sym:LIS3DH_breakout U51
@@
 NoConn ~ 9650 4050
 NoConn ~ 9750 4050
+$Comp
+L hex_master_sym:header_0.1_I2C U52
+U 1 1 5DE9837B
+P 8600 9750
+F 0 "U52" H 8828 9628 50  0000 L CNN
+F 1 "header_0.1_I2C" H 8828 9537 50  0000 L CNN
+F 2 "hex_master_board:header_0.1_i2c_12" H 8600 9950 50  0001 C CNN
+F 3 "" H 8600 9950 50  0001 C CNN
+	1    8600 9750
+	1    0    0    -1
+$EndComp
+$Comp
+L power:+5V #PWR0201
+U 1 1 5DE98A69
+P 8450 9500
+F 0 "#PWR0201" H 8450 9350 50  0001 C CNN
+F 1 "+5V" H 8465 9673 50  0000 C CNN
+F 2 "" H 8450 9500 50  0001 C CNN
+F 3 "" H 8450 9500 50  0001 C CNN
+	1    8450 9500
+	1    0    0    -1
+$EndComp
+$Comp
+L power:GND #PWR0202
+U 1 1 5DE98B84
+P 8300 9900
+F 0 "#PWR0202" H 8300 9650 50  0001 C CNN
+F 1 "GND" H 8305 9727 50  0000 C CNN
+F 2 "" H 8300 9900 50  0001 C CNN
+F 3 "" H 8300 9900 50  0001 C CNN
+	1    8300 9900
+	1    0    0    -1
+$EndComp
+Wire Wire Line
+	8550 9750 8550 9650
+Wire Wire Line
+	8550 9650 8300 9650
+Wire Wire Line
+	8300 9650 8300 9900
+Wire Wire Line
+	8450 9750 8450 9500
+Text Label 8650 9750 1    50   ~ 0
+SDA
+Text Label 8750 9750 1    50   ~ 0
+SCL
 $EndSCHEMATC

Commit message: Integrate XBEE... Functionality on first-pass PCB is done!
Parts:
- added U53: header_0.1_xbee, hex_master_board:header_0.1_xbee, symbol hex_master_sym:header_0.1_xbee
Connections:
- wire segments 430 -> 436
Changed lines of the file:
@@
 L hex_master_sym:header_0.1_I2C U52
 U 1 1 5DE9837B
-P 8600 9750
-F 0 "U52" H 8828 9628 50  0000 L CNN
-F 1 "header_0.1_I2C" H 8828 9537 50  0000 L CNN
-F 2 "hex_master_board:header_0.1_i2c_12" H 8600 9950 50  0001 C CNN
-F 3 "" H 8600 9950 50  0001 C CNN
-	1    8600 9750
+P 8500 9800
+F 0 "U52" H 8728 9678 50  0000 L CNN
+F 1 "header_0.1_I2C" H 8728 9587 50  0000 L CNN
+F 2 "hex_master_board:header_0.1_i2c_12" H 8500 10000 50  0001 C CNN
+F 3 "" H 8500 10000 50  0001 C CNN
+	1    8500 9800
 	1    0    0    -1
 $EndComp
@@
 L power:+5V #PWR0201
 U 1 1 5DE98A69
-P 8450 9500
-F 0 "#PWR0201" H 8450 9350 50  0001 C CNN
-F 1 "+5V" H 8465 9673 50  0000 C CNN
-F 2 "" H 8450 9500 50  0001 C CNN
-F 3 "" H 8450 9500 50  0001 C CNN
-	1    8450 9500
+P 8350 9550
+F 0 "#PWR0201" H 8350 9400 50  0001 C CNN
+F 1 "+5V" H 8365 9723 50  0000 C CNN
+F 2 "" H 8350 9550 50  0001 C CNN
+F 3 "" H 8350 9550 50  0001 C CNN
+	1    8350 9550
 	1    0    0    -1
 $EndComp
@@
 L power:GND #PWR0202
 U 1 1 5DE98B84
-P 8300 9900
-F 0 "#PWR0202" H 8300 9650 50  0001 C CNN
-F 1 "GND" H 8305 9727 50  0000 C CNN
-F 2 "" H 8300 9900 50  0001 C CNN
-F 3 "" H 8300 9900 50  0001 C CNN
-	1    8300 9900
+P 8200 9950
+F 0 "#PWR0202" H 8200 9700 50  0001 C CNN
+F 1 "GND" H 8205 9777 50  0000 C CNN
+F 2 "" H 8200 9950 50  0001 C CNN
+F 3 "" H 8200 9950 50  0001 C CNN
+	1    8200 9950
 	1    0    0    -1
 $EndComp
 Wire Wire Line
-	8550 9750 8550 9650
+	8450 9800 8450 9700
 Wire Wire Line
-	8550 9650 8300 9650
+	8450 9700 8200 9700
 Wire Wire Line
-	8300 9650 8300 9900
+	8200 9700 8200 9950
 Wire Wire Line
-	8450 9750 8450 9500
-Text Label 8650 9750 1    50   ~ 0
+	8350 9800 8350 9550
+Text Label 8550 9800 1    50   ~ 0
 SDA
-Text Label 8750 9750 1    50   ~ 0
+Text Label 8650 9800 1    50   ~ 0
 SCL
+$Comp
+L hex_master_sym:header_0.1_xbee U53
+U 1 1 5DF35F9C
+P 9900 9800
+F 0 "U53" H 10178 9603 50  0000 L CNN
+F 1 "header_0.1_xbee" H 10178 9512 50  0000 L CNN
+F 2 "hex_master_board:header_0.1_xbee" H 9900 9800 50  0001 C CNN
+F 3 "" H 9900 9800 50  0001 C CNN
+	1    9900 9800
+	1    0    0    -1
+$EndComp
+Text Label 10050 9850 1    50   ~ 0
+XBEE_TXD
+Text Label 9950 9850 1    50   ~ 0
+XBEE_RXD
+Wire Wire Line
+	9850 9850 9850 9700
+Wire Wire Line
+	9850 9700 9750 9700
+Wire Wire Line
+	9750 9700 9750 9600
+$Comp
+L power:+5V #PWR0203
+U 1 1 5DF9B10B
+P 9750 9600
+F 0 "#PWR0203" H 9750 9450 50  0001 C CNN
+F 1 "+5V" H 9765 9773 50  0000 C CNN
+F 2 "" H 9750 9600 50  0001 C CNN
+F 3 "" H 9750 9600 50  0001 C CNN
+	1    9750 9600
+	1    0    0    -1
+$EndComp
+$Comp
+L power:GND #PWR0204
+U 1 1 5DF9B228
+P 9500 10000
+F 0 "#PWR0204" H 9500 9750 50  0001 C CNN
+F 1 "GND" H 9505 9827 50  0000 C CNN
+F 2 "" H 9500 10000 50  0001 C CNN
+F 3 "" H 9500 10000 50  0001 C CNN
+	1    9500 10000
+	1    0    0    -1
+$EndComp
+Wire Wire Line
+	9500 10000 9500 9750
+Wire Wire Line
+	9500 9750 9750 9750
+Wire Wire Line
+	9750 9750 9750 9850
 $EndSCHEMATC

Commit message: Add silk screen labels and olin logo
Parts:
- renumbered SW1 to S0, SW2 to S1, SW11 to S10, SW12 to S11, SW3 to S2, SW4 to S3, SW5 to S4, SW6 to S5, SW7 to S6, SW8 to S7, SW9 to S8, SW10 to S9
Changed lines of the file:
@@
 	12250 2150 12250 2450
 $Comp
-L Switch:SW_DIP_x01 SW1
+L Switch:SW_DIP_x01 S0
 U 1 1 5D863B63
 P 12250 2750
-F 0 "SW1" V 11950 2800 50  0000 L CNN
+F 0 "S0" V 11950 2800 50  0000 L CNN
 F 1 "SW_DIP_x01" V 12295 2880 50  0000 L CNN
 F 2 "hex_master_board:switch_ins" H 12250 2750 50  0001 C CNN
@@
 $EndComp
 $Comp
-L Switch:SW_DIP_x01 SW2
+L Switch:SW_DIP_x01 S1
 U 1 1 5D863CF5
 P 12550 2750
-F 0 "SW2" V 12250 2800 50  0000 L CNN
+F 0 "S1" V 12250 2800 50  0000 L CNN
 F 1 "SW_DIP_x01" V 12595 2880 50  0000 L CNN
 F 2 "hex_master_board:switch_ins" H 12550 2750 50  0001 C CNN
@@
 $EndComp
 $Comp
-L Switch:SW_DIP_x01 SW3
+L Switch:SW_DIP_x01 S2
 U 1 1 5D873601
 P 12850 2750
-F 0 "SW3" V 12550 2800 50  0000 L CNN
+F 0 "S2" V 12550 2800 50  0000 L CNN
 F 1 "SW_DIP_x01" V 12895 2880 50  0000 L CNN
 F 2 "hex_master_board:switch_ins" H 12850 2750 50  0001 C CNN
@@
 $EndComp
 $Comp
-L Switch:SW_DIP_x01 SW4
+L Switch:SW_DIP_x01 S3
 U 1 1 5D882F0E
 P 13150 2750
-F 0 "SW4" V 12850 2800 50  0000 L CNN
+F 0 "S3" V 12850 2800 50  0000 L CNN
 F 1 "SW_DIP_x01" V 13195 2880 50  0000 L CNN
 F 2 "hex_master_board:switch_ins" H 13150 2750 50  0001 C CNN
@@
 $EndComp
 $Comp
-L Switch:SW_DIP_x01 SW5
+L Switch:SW_DIP_x01 S4
 U 1 1 5D89281A
 P 13450 2750
-F 0 "SW5" V 13150 2800 50  0000 L CNN
+F 0 "S4" V 13150 2800 50  0000 L CNN
 F 1 "SW_DIP_x01" V 13495 2880 50  0000 L CNN
 F 2 "hex_master_board:switch_ins" H 13450 2750 50  0001 C CNN
@@
 $EndComp
 $Comp
-L Switch:SW_DIP_x01 SW6
+L Switch:SW_DIP_x01 S5
 U 1 1 5D8A2129
 P 13750 2750
-F 0 "SW6" V 13450 2800 50  0000 L CNN
+F 0 "S5" V 13450 2800 50  0000 L CNN
 F 1 "SW_DIP_x01" V 13795 2880 50  0000 L CNN
 F 2 "hex_master_board:switch_ins" H 13750 2750 50  0001 C CNN
@@
 	14050 2150 14050 2450
 $Comp
-L Switch:SW_DIP_x01 SW7
+L Switch:SW_DIP_x01 S6
 U 1 1 5DB26DC7
 P 14050 2750
-F 0 "SW7" V 13750 2800 50  0000 L CNN
+F 0 "S6" V 13750 2800 50  0000 L CNN
 F 1 "SW_DIP_x01" V 14095 2880 50  0000 L CNN
 F 2 "hex_master_board:switch_ins" H 14050 2750 50  0001 C CNN
@@
 $EndComp
 $Comp
-L Switch:SW_DIP_x01 SW8
+L Switch:SW_DIP_x01 S7
 U 1 1 5DB26DCE
 P 14350 2750
-F 0 "SW8" V 14050 2800 50  0000 L CNN
+F 0 "S7" V 14050 2800 50  0000 L CNN
 F 1 "SW_DIP_x01" V 14395 2880 50  0000 L CNN
 F 2 "hex_master_board:switch_ins" H 14350 2750 50  0001 C CNN
@@
 $EndComp
 $Comp
-L Switch:SW_DIP_x01 SW9
+L Switch:SW_DIP_x01 S8
 U 1 1 5DB26DD5
 P 14650 2750
-F 0 "SW9" V 14350 2800 50  0000 L CNN
+F 0 "S8" V 14350 2800 50  0000 L CNN
 F 1 "SW_DIP_x01" V 14695 2880 50  0000 L CNN
 F 2 "hex_master_board:switch_ins" H 14650 2750 50  0001 C CNN
@@
 $EndComp
 $Comp
-L Switch:SW_DIP_x01 SW10
+L Switch:SW_DIP_x01 S9
 U 1 1 5DB26DDC
 P 14950 2750
-F 0 "SW10" V 14650 2800 50  0000 L CNN
+F 0 "S9" V 14650 2800 50  0000 L CNN
 F 1 "SW_DIP_x01" V 14995 2880 50  0000 L CNN
 F 2 "hex_master_board:switch_ins" H 14950 2750 50  0001 C CNN
@@
 $EndComp
 $Comp
-L Switch:SW_DIP_x01 SW11
+L Switch:SW_DIP_x01 S10
 U 1 1 5DB26DE3
 P 15250 2750
-F 0 "SW11" V 14950 2800 50  0000 L CNN
+F 0 "S10" V 14950 2800 50  0000 L CNN
 F 1 "SW_DIP_x01" V 15295 2880 50  0000 L CNN
 F 2 "hex_master_board:switch_ins" H 15250 2750 50  0001 C CNN
@@
 $EndComp
 $Comp
-L Switch:SW_DIP_x01 SW12
+L Switch:SW_DIP_x01 S11
 U 1 1 5DB26DEA
 P 15550 2750
-F 0 "SW12" V 15250 2800 50  0000 L CNN
+F 0 "S11" V 15250 2800 50  0000 L CNN
 F 1 "SW_DIP_x01" V 15595 2880 50  0000 L CNN
 F 2 "hex_master_board:switch_ins" H 15550 2750 50  0001 C CNN
